File: pcb/MIDI Mixer One.sch (KiCad schematic (older format))
At the start: 65 parts, among them SW1 SW_Push, SW10 SW_Push, SW11 SW_Push, SW12 SW_Push, SW2 SW_Push, SW3 SW_Push, SW4 SW_Push, SW5 SW_Push, SW6 SW_Push, SW7 SW_Push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

Commit message: cleanup kicad libs and cache files
Parts:
- U1: symbol MIDI-Mixer-One-rescue:Teensy-LC-Teensy-MIDI-Mixer-One-v01-rescue -> Teensy:Teensy-LC
Changed lines of the file:
@@
 $EndComp
 $Comp
-L MIDI-Mixer-One-rescue:Teensy-LC-Teensy-MIDI-Mixer-One-v01-rescue U1
+L Teensy:Teensy-LC U1
 U 1 1 5EBE1898
 P 4200 8300
